Commit message: finally fixing the hack of new_gazebo_version to set root joint for pinocchio as per robot_control commit fccb58b1fb819f6c18701ba5d1a20bd6d21af330

File: robots/aliengo.urdf.xacro (robot description, xacro)
@@ -7,5 +7,4 @@
     <xacro:arg name="arm_enabled" default="false"/>
     <xacro:arg name="arm_name" default="kinova"/>
-    <xacro:arg name="new_gazebo_version" default="false"/>
     <xacro:arg name="robot_name"  default="aliengo"/>
     <xacro:arg name="base_name"   default="trunk"/>
@@ -25,13 +24,4 @@
     <!-- Rollover Protection mode will add an additional stick on the top, use "true" or "false" to switch it. -->
     <xacro:property name="rolloverProtection" value="false"/>
-    <!-- Floating-base Joint -->
-    <xacro:unless value="$(arg new_gazebo_version)">
-            <link name="world"/>
-            <joint name="floating_base_joint" type="floating">
-              <origin rpy="0 0 0" xyz="0 0 0"/>
-              <parent link="world"/>
-              <child link="base_link"/>
-            </joint>
-    </xacro:unless>
     <link name="base_link" />
    <joint name="floating_base" type="fixed">
